File: hardware/desklight.sch (KiCad schematic (older format))
At the start: 10 parts, among them IC1 ATTINY10-TS, P1 AVR_TPI, P2 Pwr5V1500mA, P3 WS2812_CON, SW1 COLOR_SW

Commit message: reduce flickering: hardware improvement, IIR filter for ADC; use more dynamic of potentiometer
Parts:
- removed C?: 10u, symbol CP1
- added C1: C, symbol C
- added C2: 10p, symbol C
- renumbered C2 to C3, C3 to C4
Connections:
- wire segments 34 -> 36
Other:
- moved on the sheet: P2, R1
Changed lines of the file:
@@
 $EndComp
 $Comp
-L C C3
+L C C4
 U 1 1 588C115D
 P 9700 3950
-F 0 "C3" H 9725 4050 50  0000 L CNN
+F 0 "C4" H 9725 4050 50  0000 L CNN
 F 1 "100n" H 9725 3850 50  0000 L CNN
 F 2 "" H 9738 3800 50  0000 C CNN
@@
 $EndComp
 $Comp
-L VCC #PWR01
+L VCC #PWR12
 U 1 1 588C121F
 P 9700 3550
-F 0 "#PWR01" H 9700 3400 50  0001 C CNN
+F 0 "#PWR12" H 9700 3400 50  0001 C CNN
 F 1 "VCC" H 9700 3700 50  0000 C CNN
 F 2 "" H 9700 3550 50  0000 C CNN
@@
 $EndComp
 $Comp
-L GND #PWR02
+L GND #PWR13
 U 1 1 588C1246
 P 9700 4350
-F 0 "#PWR02" H 9700 4100 50  0001 C CNN
+F 0 "#PWR13" H 9700 4100 50  0001 C CNN
 F 1 "GND" H 9700 4200 50  0000 C CNN
 F 2 "" H 9700 4350 50  0000 C CNN
@@
 L CONN_01X02 P2
 U 1 1 588C12C5
-P 2150 2250
-F 0 "P2" H 2150 2400 50  0000 C CNN
-F 1 "Pwr5V1500mA" V 2250 2250 50  0000 C CNN
-F 2 "" H 2150 2250 50  0000 C CNN
-F 3 "" H 2150 2250 50  0000 C CNN
-	1    2150 2250
+P 2200 2250
+F 0 "P2" H 2200 2400 50  0000 C CNN
+F 1 "Pwr5V1500mA" V 2300 2250 50  0000 C CNN
+F 2 "" H 2200 2250 50  0000 C CNN
+F 3 "" H 2200 2250 50  0000 C CNN
+	1    2200 2250
 	1    0    0    1
 $EndComp
 $Comp
-L PWR_FLAG #FLG03
+L PWR_FLAG #FLG1
 U 1 1 588C1337
-P 1850 2100
-F 0 "#FLG03" H 1850 2195 50  0001 C CNN
-F 1 "PWR_FLAG" H 1850 2280 50  0000 C CNN
-F 2 "" H 1850 2100 50  0000 C CNN
-F 3 "" H 1850 2100 50  0000 C CNN
-	1    1850 2100
-	1    0    0    -1
-$EndComp
-$Comp
-L PWR_FLAG #FLG04
+P 1650 1900
+F 0 "#FLG1" H 1650 1995 50  0001 C CNN
+F 1 "PWR_FLAG" H 1650 2080 50  0000 C CNN
+F 2 "" H 1650 1900 50  0000 C CNN
+F 3 "" H 1650 1900 50  0000 C CNN
+	1    1650 1900
+	1    0    0    -1
+$EndComp
+$Comp
+L PWR_FLAG #FLG2
 U 1 1 588C135A
-P 1850 2400
-F 0 "#FLG04" H 1850 2495 50  0001 C CNN
-F 1 "PWR_FLAG" H 1850 2580 50  0000 C CNN
-F 2 "" H 1850 2400 50  0000 C CNN
-F 3 "" H 1850 2400 50  0000 C CNN
-	1    1850 2400
+P 1650 2600
+F 0 "#FLG2" H 1650 2695 50  0001 C CNN
+F 1 "PWR_FLAG" H 1650 2780 50  0000 C CNN
+F 2 "" H 1650 2600 50  0000 C CNN
+F 3 "" H 1650 2600 50  0000 C CNN
+	1    1650 2600
 	-1   0    0    1
 $EndComp
 $Comp
-L GND #PWR05
+L GND #PWR2
 U 1 1 588C1377
-P 1500 2400
-F 0 "#PWR05" H 1500 2150 50  0001 C CNN
-F 1 "GND" H 1500 2250 50  0000 C CNN
-F 2 "" H 1500 2400 50  0000 C CNN
-F 3 "" H 1500 2400 50  0000 C CNN
-	1    1500 2400
-	1    0    0    -1
-$EndComp
-$Comp
-L VCC #PWR06
+P 1300 2600
+F 0 "#PWR2" H 1300 2350 50  0001 C CNN
+F 1 "GND" H 1300 2450 50  0000 C CNN
+F 2 "" H 1300 2600 50  0000 C CNN
+F 3 "" H 1300 2600 50  0000 C CNN
+	1    1300 2600
+	1    0    0    -1
+$EndComp
+$Comp
+L VCC #PWR1
 U 1 1 588C1394
-P 1500 2100
-F 0 "#PWR06" H 1500 1950 50  0001 C CNN
-F 1 "VCC" H 1500 2250 50  0000 C CNN
-F 2 "" H 1500 2100 50  0000 C CNN
-F 3 "" H 1500 2100 50  0000 C CNN
-	1    1500 2100
+P 1300 1900
+F 0 "#PWR1" H 1300 1750 50  0001 C CNN
+F 1 "VCC" H 1300 2050 50  0000 C CNN
+F 2 "" H 1300 1900 50  0000 C CNN
+F 3 "" H 1300 1900 50  0000 C CNN
+	1    1300 1900
 	1    0    0    -1
 $EndComp
@@
 $EndComp
 $Comp
-L VCC #PWR07
+L VCC #PWR3
 U 1 1 588C14B1
 P 2300 5800
-F 0 "#PWR07" H 2300 5650 50  0001 C CNN
+F 0 "#PWR3" H 2300 5650 50  0001 C CNN
 F 1 "VCC" H 2300 5950 50  0000 C CNN
 F 2 "" H 2300 5800 50  0000 C CNN
@@
 $EndComp
 $Comp
-L GND #PWR08
+L GND #PWR4
 U 1 1 588C14D1
 P 2300 6200
-F 0 "#PWR08" H 2300 5950 50  0001 C CNN
+F 0 "#PWR4" H 2300 5950 50  0001 C CNN
 F 1 "GND" H 2300 6050 50  0000 C CNN
 F 2 "" H 2300 6200 50  0000 C CNN
@@
 $EndComp
 $Comp
-L GND #PWR09
+L GND #PWR8
 U 1 1 588C17B4
 P 6100 3200
-F 0 "#PWR09" H 6100 2950 50  0001 C CNN
+F 0 "#PWR8" H 6100 2950 50  0001 C CNN
 F 1 "GND" H 6100 3050 50  0000 C CNN
 F 2 "" H 6100 3200 50  0000 C CNN
@@
 $EndComp
 $Comp
-L VCC #PWR010
+L VCC #PWR10
 U 1 1 588C1829
 P 6400 3200
-F 0 "#PWR010" H 6400 3050 50  0001 C CNN
+F 0 "#PWR10" H 6400 3050 50  0001 C CNN
 F 1 "VCC" H 6400 3350 50  0000 C CNN
 F 2 "" H 6400 3200 50  0000 C CNN
@@
 $EndComp
 $Comp
-L GND #PWR011
+L GND #PWR11
 U 1 1 588C1BAB
 P 6500 4800
-F 0 "#PWR011" H 6500 4550 50  0001 C CNN
+F 0 "#PWR11" H 6500 4550 50  0001 C CNN
 F 1 "GND" H 6500 4650 50  0000 C CNN
 F 2 "" H 6500 4800 50  0000 C CNN
@@
 $EndComp
 $Comp
-L C C2
+L C C3
 U 1 1 588C1BF7
 P 6100 4400
-F 0 "C2" H 6125 4500 50  0000 L CNN
+F 0 "C3" H 6125 4500 50  0000 L CNN
 F 1 "100n" H 6125 4300 50  0000 L CNN
 F 2 "" H 6138 4250 50  0000 C CNN
@@
 	1    0    0    -1
 $EndComp
-Wire Wire Line
-	9500 3700 9700 3700
-Wire Wire Line
-	9700 3550 9700 3800
-Wire Wire Line
-	9700 4100 9700 4350
-Wire Wire Line
-	9700 4200 9500 4200
-Connection ~ 9700 3700
-Connection ~ 9700 4200
-Wire Wire Line
-	1500 2100 1500 2200
-Wire Wire Line
-	1500 2200 1950 2200
-Wire Wire Line
-	1850 2200 1850 2100
-Connection ~ 1850 2200
-Wire Wire Line
-	1500 2400 1500 2300
-Wire Wire Line
-	1500 2300 1950 2300
-Wire Wire Line
-	1850 2400 1850 2300
-Connection ~ 1850 2300
-Wire Wire Line
-	2200 5900 2300 5900
-Wire Wire Line
-	2300 5900 2300 5800
-Wire Wire Line
-	2200 6100 2300 6100
-Wire Wire Line
-	2300 6100 2300 6200
-Wire Wire Line
-	1700 5900 1400 5900
-Wire Wire Line
-	1700 6000 1400 6000
-Wire Wire Line
-	1700 6100 1400 6100
-Wire Wire Line
-	5850 3900 7100 3900
-Wire Wire Line
-	7100 4100 6800 4100
-Wire Wire Line
-	6100 3100 6100 3200
-Wire Wire Line
-	6300 3100 6300 3200
-Wire Wire Line
-	6300 3200 6400 3200
-Wire Wire Line
-	6100 4000 7100 4000
-Wire Wire Line
-	6500 4000 6500 4100
-Wire Wire Line
-	6100 4000 6100 4250
-Connection ~ 6500 4000
-Wire Wire Line
-	6100 4550 6100 4800
-Wire Wire Line
-	6500 4800 6500 4700
 $Comp
 L POT RV1
@@
 $EndComp
 $Comp
-L VCC #PWR012
+L VCC #PWR5
 U 1 1 588C225B
 P 4950 3600
-F 0 "#PWR012" H 4950 3450 50  0001 C CNN
+F 0 "#PWR5" H 4950 3450 50  0001 C CNN
 F 1 "VCC" H 4950 3750 50  0000 C CNN
 F 2 "" H 4950 3600 50  0000 C CNN
@@
 	1    0    0    -1
 $EndComp
-Wire Wire Line
-	4950 3600 4950 3750
-$Comp
-L GND #PWR013
+$Comp
+L GND #PWR6
 U 1 1 588C22B6
 P 4950 4800
-F 0 "#PWR013" H 4950 4550 50  0001 C CNN
+F 0 "#PWR6" H 4950 4550 50  0001 C CNN
 F 1 "GND" H 4950 4650 50  0000 C CNN
 F 2 "" H 4950 4800 50  0000 C CNN
@@
 	1    0    0    -1
 $EndComp
-Wire Wire Line
-	4950 4800 4950 4050
-Wire Wire Line
-	6200 3100 6200 3800
-Wire Wire Line
-	6200 3800 7100 3800
 $Comp
 L R R1
 U 1 1 588C284D
-P 5700 3900
-F 0 "R1" V 5780 3900 50  0000 C CNN
-F 1 "470" V 5700 3900 50  0000 C CNN
-F 2 "" V 5630 3900 50  0000 C CNN
-F 3 "" H 5700 3900 50  0000 C CNN
-	1    5700 3900
+P 5350 3900
+F 0 "R1" V 5430 3900 50  0000 C CNN
+F 1 "470" V 5350 3900 50  0000 C CNN
+F 2 "" V 5280 3900 50  0000 C CNN
+F 3 "" H 5350 3900 50  0000 C CNN
+	1    5350 3900
 	0    1    1    0
 $EndComp
-Wire Wire Line
-	5100 3900 5550 3900
-Wire Wire Line
-	5300 3900 5300 4250
-Connection ~ 5300 3900
-$Comp
-L GND #PWR014
+$Comp
+L GND #PWR7
 U 1 1 588C2BCF
-P 5300 4800
-F 0 "#PWR014" H 5300 4550 50  0001 C CNN
-F 1 "GND" H 5300 4650 50  0000 C CNN
-F 2 "" H 5300 4800 50  0000 C CNN
-F 3 "" H 5300 4800 50  0000 C CNN
-	1    5300 4800
-	1    0    0    -1
-$EndComp
-Wire Wire Line
-	5300 4800 5300 4550
-$Comp
-L GND #PWR015
+P 5700 4800
+F 0 "#PWR7" H 5700 4550 50  0001 C CNN
+F 1 "GND" H 5700 4650 50  0000 C CNN
+F 2 "" H 5700 4800 50  0000 C CNN
+F 3 "" H 5700 4800 50  0000 C CNN
+	1    5700 4800
+	1    0    0    -1
+$EndComp
+$Comp
+L GND #PWR9
 U 1 1 588C2C7A
 P 6100 4800
-F 0 "#PWR015" H 6100 4550 50  0001 C CNN
+F 0 "#PWR9" H 6100 4550 50  0001 C CNN
 F 1 "GND" H 6100 4650 50  0000 C CNN
 F 2 "" H 6100 4800 50  0000 C CNN
@@
 	1    0    0    -1
 $EndComp
+Text Label 6200 3450 3    60   ~ 0
+DOUT
+$Comp
+L C C1
+U 1 1 588D4639
+P 1300 2250
+F 0 "C1" H 1325 2350 50  0000 L CNN
+F 1 "C" H 1325 2150 50  0000 L CNN
+F 2 "" H 1338 2100 50  0000 C CNN
+F 3 "" H 1300 2250 50  0000 C CNN
+	1    1300 2250
+	1    0    0    -1
+$EndComp
+Wire Wire Line
+	9500 3700 9700 3700
+Wire Wire Line
+	9700 3550 9700 3800
+Wire Wire Line
+	9700 4100 9700 4350
+Wire Wire Line
+	9700 4200 9500 4200
+Connection ~ 9700 3700
+Connection ~ 9700 4200
+Wire Wire Line
+	2200 5900 2300 5900
+Wire Wire Line
+	2300 5900 2300 5800
+Wire Wire Line
+	2200 6100 2300 6100
+Wire Wire Line
+	2300 6100 2300 6200
+Wire Wire Line
+	1700 5900 1400 5900
+Wire Wire Line
+	1700 6000 1400 6000
+Wire Wire Line
+	1700 6100 1400 6100
+Wire Wire Line
+	5500 3900 7100 3900
+Wire Wire Line
+	7100 4100 6800 4100
+Wire Wire Line
+	6100 3100 6100 3200
+Wire Wire Line
+	6300 3100 6300 3200
+Wire Wire Line
+	6300 3200 6400 3200
+Wire Wire Line
+	6100 4000 7100 4000
+Wire Wire Line
+	6500 4000 6500 4100
+Wire Wire Line
+	6100 4000 6100 4250
+Connection ~ 6500 4000
+Wire Wire Line
+	6100 4550 6100 4800
+Wire Wire Line
+	6500 4800 6500 4700
+Wire Wire Line
+	4950 3600 4950 3750
+Wire Wire Line
+	4950 4800 4950 4050
+Wire Wire Line
+	6200 3100 6200 3800
+Wire Wire Line
+	6200 3800 7100 3800
+Wire Wire Line
+	5100 3900 5200 3900
+Wire Wire Line
+	5700 4800 5700 4550
 Wire Notes Line
 	3350 500  3350 7750
 Wire Notes Line
 	3350 4000 500  4000
-Text Label 6200 3450 3    60   ~ 0
-DOUT
-$Comp
-L CP1 C?
-U 1 1 588C4485
-P 5300 4400
-F 0 "C?" H 5325 4500 50  0000 L CNN
-F 1 "10u" H 5325 4300 50  0000 L CNN
-F 2 "" H 5300 4400 50  0000 C CNN
-F 3 "" H 5300 4400 50  0000 C CNN
-	1    5300 4400
-	1    0    0    -1
-$EndComp
+Wire Wire Line
+	1300 1900 1300 2100
+Wire Wire Line
+	1300 2400 1300 2600
+Wire Wire Line
+	1300 2500 1650 2500
+Wire Wire Line
+	1650 2300 1650 2600
+Connection ~ 1300 2500
+Wire Wire Line
+	1300 2000 1650 2000
+Wire Wire Line
+	1650 1900 1650 2200
+Connection ~ 1300 2000
+Wire Wire Line
+	1650 2200 2000 2200
+Connection ~ 1650 2000
+Wire Wire Line
+	1650 2300 2000 2300
+Connection ~ 1650 2500
+Wire Wire Line
+	5700 4250 5700 3900
+Connection ~ 5700 3900
+$Comp
+L C C2
+U 1 1 588D4AD7
+P 5700 4400
+F 0 "C2" H 5725 4500 50  0000 L CNN
+F 1 "10p" H 5725 4300 50  0000 L CNN
+F 2 "" H 5738 4250 50  0000 C CNN
+F 3 "" H 5700 4400 50  0000 C CNN
+	1    5700 4400
+	1    0    0    -1
+$EndComp

Commit message: initial refactor and preps for encoder use
Parts:
- removed R1: 470, symbol R
- removed RV1: 50k, symbol POT
- removed SW1: COLOR_SW, symbol SW_PUSH
- added C3: 100n, symbol C
- added SW1: Rotary_Encoder_Switch, symbol Rotary_Encoder_Switch
- C2: value 10p -> 100n
- renumbered C3 to C4, C4 to C5
Connections:
- wire segments 36 -> 40
Other:
- moved on the sheet: C4
Changed lines of the file:
@@
 EESchema Schematic File Version 2
+LIBS:desklight-rescue
 LIBS:power
 LIBS:device
@@
 $EndComp
 $Comp
-L C C4
+L C C5
 U 1 1 588C115D
 P 9700 3950
-F 0 "C4" H 9725 4050 50  0000 L CNN
+F 0 "C5" H 9725 4050 50  0000 L CNN
 F 1 "100n" H 9725 3850 50  0000 L CNN
 F 2 "" H 9738 3800 50  0000 C CNN
@@
 $EndComp
 $Comp
-L VCC #PWR12
+L VCC #PWR01
 U 1 1 588C121F
 P 9700 3550
-F 0 "#PWR12" H 9700 3400 50  0001 C CNN
+F 0 "#PWR01" H 9700 3400 50  0001 C CNN
 F 1 "VCC" H 9700 3700 50  0000 C CNN
 F 2 "" H 9700 3550 50  0000 C CNN
@@
 $EndComp
 $Comp
-L GND #PWR13
+L GND #PWR02
 U 1 1 588C1246
 P 9700 4350
-F 0 "#PWR13" H 9700 4100 50  0001 C CNN
+F 0 "#PWR02" H 9700 4100 50  0001 C CNN
 F 1 "GND" H 9700 4200 50  0000 C CNN
 F 2 "" H 9700 4350 50  0000 C CNN
@@
 $EndComp
 $Comp
-L PWR_FLAG #FLG1
+L PWR_FLAG #FLG03
 U 1 1 588C1337
 P 1650 1900
-F 0 "#FLG1" H 1650 1995 50  0001 C CNN
+F 0 "#FLG03" H 1650 1995 50  0001 C CNN
 F 1 "PWR_FLAG" H 1650 2080 50  0000 C CNN
 F 2 "" H 1650 1900 50  0000 C CNN
@@
 $EndComp
 $Comp
-L PWR_FLAG #FLG2
+L PWR_FLAG #FLG04
 U 1 1 588C135A
 P 1650 2600
-F 0 "#FLG2" H 1650 2695 50  0001 C CNN
+F 0 "#FLG04" H 1650 2695 50  0001 C CNN
 F 1 "PWR_FLAG" H 1650 2780 50  0000 C CNN
 F 2 "" H 1650 2600 50  0000 C CNN
@@
 $EndComp
 $Comp
-L GND #PWR2
+L GND #PWR05
 U 1 1 588C1377
 P 1300 2600
-F 0 "#PWR2" H 1300 2350 50  0001 C CNN
+F 0 "#PWR05" H 1300 2350 50  0001 C CNN
 F 1 "GND" H 1300 2450 50  0000 C CNN
 F 2 "" H 1300 2600 50  0000 C CNN
@@
 $EndComp
 $Comp
-L VCC #PWR1
+L VCC #PWR06
 U 1 1 588C1394
 P 1300 1900
-F 0 "#PWR1" H 1300 1750 50  0001 C CNN
+F 0 "#PWR06" H 1300 1750 50  0001 C CNN
 F 1 "VCC" H 1300 2050 50  0000 C CNN
 F 2 "" H 1300 1900 50  0000 C CNN
@@
 $EndComp
 $Comp
-L VCC #PWR3
+L VCC #PWR07
 U 1 1 588C14B1
 P 2300 5800
-F 0 "#PWR3" H 2300 5650 50  0001 C CNN
+F 0 "#PWR07" H 2300 5650 50  0001 C CNN
 F 1 "VCC" H 2300 5950 50  0000 C CNN
 F 2 "" H 2300 5800 50  0000 C CNN
@@
 $EndComp
 $Comp
-L GND #PWR4
+L GND #PWR08
 U 1 1 588C14D1
 P 2300 6200
-F 0 "#PWR4" H 2300 5950 50  0001 C CNN
+F 0 "#PWR08" H 2300 5950 50  0001 C CNN
 F 1 "GND" H 2300 6050 50  0000 C CNN
 F 2 "" H 2300 6200 50  0000 C CNN
@@
 $EndComp
 $Comp
-L GND #PWR8
+L GND #PWR09
 U 1 1 588C17B4
 P 6100 3200
-F 0 "#PWR8" H 6100 2950 50  0001 C CNN
+F 0 "#PWR09" H 6100 2950 50  0001 C CNN
 F 1 "GND" H 6100 3050 50  0000 C CNN
 F 2 "" H 6100 3200 50  0000 C CNN
@@
 $EndComp
 $Comp
-L VCC #PWR10
+L VCC #PWR010
 U 1 1 588C1829
 P 6400 3200
-F 0 "#PWR10" H 6400 3050 50  0001 C CNN
+F 0 "#PWR010" H 6400 3050 50  0001 C CNN
 F 1 "VCC" H 6400 3350 50  0000 C CNN
 F 2 "" H 6400 3200 50  0000 C CNN
@@
 $EndComp
 $Comp
-L SW_PUSH SW1
-U 1 1 588C1AB7
-P 6500 4400
-F 0 "SW1" H 6650 4510 50  0000 C CNN
-F 1 "COLOR_SW" H 6500 4320 50  0000 C CNN
-F 2 "" H 6500 4400 50  0000 C CNN
-F 3 "" H 6500 4400 50  0000 C CNN
-	1    6500 4400
-	0    1    1    0
-$EndComp
-$Comp
-L GND #PWR11
+L GND #PWR011
 U 1 1 588C1BAB
-P 6500 4800
-F 0 "#PWR11" H 6500 4550 50  0001 C CNN
-F 1 "GND" H 6500 4650 50  0000 C CNN
-F 2 "" H 6500 4800 50  0000 C CNN
-F 3 "" H 6500 4800 50  0000 C CNN
-	1    6500 4800
-	1    0    0    -1
-$EndComp
-$Comp
-L C C3
+P 6450 5000
+F 0 "#PWR011" H 6450 4750 50  0001 C CNN
+F 1 "GND" H 6450 4850 50  0000 C CNN
+F 2 "" H 6450 5000 50  0000 C CNN
+F 3 "" H 6450 5000 50  0000 C CNN
+	1    6450 5000
+	1    0    0    -1
+$EndComp
+$Comp
+L C C4
 U 1 1 588C1BF7
-P 6100 4400
-F 0 "C3" H 6125 4500 50  0000 L CNN
-F 1 "100n" H 6125 4300 50  0000 L CNN
-F 2 "" H 6138 4250 50  0000 C CNN
-F 3 "" H 6100 4400 50  0000 C CNN
-	1    6100 4400
-	1    0    0    -1
-$EndComp
-$Comp
-L POT RV1
-U 1 1 588C21B8
-P 4950 3900
-F 0 "RV1" H 4950 3820 50  0000 C CNN
-F 1 "50k" H 4950 3900 50  0000 C CNN
-F 2 "" H 4950 3900 50  0000 C CNN
-F 3 "" H 4950 3900 50  0000 C CNN
-	1    4950 3900
-	0    1    -1   0
-$EndComp
-$Comp
-L VCC #PWR5
-U 1 1 588C225B
-P 4950 3600
-F 0 "#PWR5" H 4950 3450 50  0001 C CNN
-F 1 "VCC" H 4950 3750 50  0000 C CNN
-F 2 "" H 4950 3600 50  0000 C CNN
-F 3 "" H 4950 3600 50  0000 C CNN
-	1    4950 3600
-	1    0    0    -1
-$EndComp
-$Comp
-L GND #PWR6
-U 1 1 588C22B6
-P 4950 4800
-F 0 "#PWR6" H 4950 4550 50  0001 C CNN
-F 1 "GND" H 4950 4650 50  0000 C CNN
-F 2 "" H 4950 4800 50  0000 C CNN
-F 3 "" H 4950 4800 50  0000 C CNN
-	1    4950 4800
-	1    0    0    -1
-$EndComp
-$Comp
-L R R1
-U 1 1 588C284D
-P 5350 3900
-F 0 "R1" V 5430 3900 50  0000 C CNN
-F 1 "470" V 5350 3900 50  0000 C CNN
-F 2 "" V 5280 3900 50  0000 C CNN
-F 3 "" H 5350 3900 50  0000 C CNN
-	1    5350 3900
-	0    1    1    0
-$EndComp
-$Comp
-L GND #PWR7
-U 1 1 588C2BCF
-P 5700 4800
-F 0 "#PWR7" H 5700 4550 50  0001 C CNN
-F 1 "GND" H 5700 4650 50  0000 C CNN
-F 2 "" H 5700 4800 50  0000 C CNN
-F 3 "" H 5700 4800 50  0000 C CNN
-	1    5700 4800
-	1    0    0    -1
-$EndComp
-$Comp
-L GND #PWR9
+P 6700 4750
+F 0 "C4" H 6725 4850 50  0000 L CNN
+F 1 "100n" H 6725 4650 50  0000 L CNN
+F 2 "" H 6738 4600 50  0000 C CNN
+F 3 "" H 6700 4750 50  0000 C CNN
+	1    6700 4750
+	1    0    0    -1
+$EndComp
+$Comp
+L GND #PWR012
 U 1 1 588C2C7A
-P 6100 4800
-F 0 "#PWR9" H 6100 4550 50  0001 C CNN
-F 1 "GND" H 6100 4650 50  0000 C CNN
-F 2 "" H 6100 4800 50  0000 C CNN
-F 3 "" H 6100 4800 50  0000 C CNN
-	1    6100 4800
+P 6700 5000
+F 0 "#PWR012" H 6700 4750 50  0001 C CNN
+F 1 "GND" H 6700 4850 50  0000 C CNN
+F 2 "" H 6700 5000 50  0000 C CNN
+F 3 "" H 6700 5000 50  0000 C CNN
+	1    6700 5000
 	1    0    0    -1
 $EndComp
@@
 	1    0    0    -1
 $EndComp
+$Comp
+L Rotary_Encoder_Switch SW1
+U 1 1 58C9CC1D
+P 5950 4400
+F 0 "SW1" H 5950 4660 50  0000 C CNN
+F 1 "Rotary_Encoder_Switch" H 5950 4140 50  0000 C CNN
+F 2 "" H 5850 4560 50  0001 C CNN
+F 3 "" H 5950 4660 50  0001 C CNN
+	1    5950 4400
+	1    0    0    -1
+$EndComp
 Wire Wire Line
 	9500 3700 9700 3700
@@
 	1700 6100 1400 6100
 Wire Wire Line
-	5500 3900 7100 3900
-Wire Wire Line
-	7100 4100 6800 4100
+	6700 4100 7100 4100
 Wire Wire Line
 	6100 3100 6100 3200
@@
 	6300 3200 6400 3200
 Wire Wire Line
-	6100 4000 7100 4000
-Wire Wire Line
-	6500 4000 6500 4100
-Wire Wire Line
-	6100 4000 6100 4250
-Connection ~ 6500 4000
-Wire Wire Line
-	6100 4550 6100 4800
-Wire Wire Line
-	6500 4800 6500 4700
-Wire Wire Line
-	4950 3600 4950 3750
-Wire Wire Line
-	4950 4800 4950 4050
-Wire Wire Line
 	6200 3100 6200 3800
 Wire Wire Line
 	6200 3800 7100 3800
-Wire Wire Line
-	5100 3900 5200 3900
-Wire Wire Line
-	5700 4800 5700 4550
 Wire Notes Line
 	3350 500  3350 7750
@@
 Connection ~ 1650 2500
 Wire Wire Line
-	5700 4250 5700 3900
-Connection ~ 5700 3900
+	6250 4500 6450 4500
+Wire Wire Line
+	6450 4500 6450 5000
+Wire Wire Line
+	6250 4300 6700 4300
+Wire Wire Line
+	6700 4100 6700 4600
+Wire Wire Line
+	6700 5000 6700 4900
+Wire Wire Line
+	4800 3900 7100 3900
+Connection ~ 6700 4300
+Wire Wire Line
+	7100 4000 5100 4000
+Wire Wire Line
+	5100 4000 5100 4600
+Wire Wire Line
+	5100 4300 5650 4300
+Wire Wire Line
+	4800 3900 4800 4600
+Wire Wire Line
+	4800 4500 5650 4500
+Wire Wire Line
+	5650 4400 5400 4400
 $Comp
 L C C2
-U 1 1 588D4AD7
-P 5700 4400
-F 0 "C2" H 5725 4500 50  0000 L CNN
-F 1 "10p" H 5725 4300 50  0000 L CNN
-F 2 "" H 5738 4250 50  0000 C CNN
-F 3 "" H 5700 4400 50  0000 C CNN
-	1    5700 4400
-	1    0    0    -1
-$EndComp
+U 1 1 58C9DD44
+P 4800 4750
+F 0 "C2" H 4825 4850 50  0000 L CNN
+F 1 "100n" H 4825 4650 50  0000 L CNN
+F 2 "" H 4838 4600 50  0000 C CNN
+F 3 "" H 4800 4750 50  0000 C CNN
+	1    4800 4750
+	1    0    0    -1
+$EndComp
+$Comp
+L C C3
+U 1 1 58C9DDBA
+P 5100 4750
+F 0 "C3" H 5125 4850 50  0000 L CNN
+F 1 "100n" H 5125 4650 50  0000 L CNN
+F 2 "" H 5138 4600 50  0000 C CNN
+F 3 "" H 5100 4750 50  0000 C CNN
+	1    5100 4750
+	1    0    0    -1
+$EndComp
+Connection ~ 5100 4300
+Connection ~ 4800 4500
+Wire Wire Line
+	4800 4900 4800 5000
+$Comp
+L GND #PWR013
+U 1 1 58C9E040
+P 5100 5000
+F 0 "#PWR013" H 5100 4750 50  0001 C CNN
+F 1 "GND" H 5100 4850 50  0000 C CNN
+F 2 "" H 5100 5000 50  0000 C CNN
+F 3 "" H 5100 5000 50  0000 C CNN
+	1    5100 5000
+	1    0    0    -1
+$EndComp
+Wire Wire Line
+	5100 5000 5100 4900
+$Comp
+L GND #PWR015
+U 1 1 58C9ED0D
+P 4800 5000
+F 0 "#PWR015" H 4800 4750 50  0001 C CNN
+F 1 "GND" H 4800 4850 50  0000 C CNN
+F 2 "" H 4800 5000 50  0000 C CNN
+F 3 "" H 4800 5000 50  0000 C CNN
+	1    4800 5000
+	1    0    0    -1
+$EndComp
+$Comp
+L GND #PWR014
+U 1 1 58C9ECDB
+P 5400 5000
+F 0 "#PWR014" H 5400 4750 50  0001 C CNN
+F 1 "GND" H 5400 4850 50  0000 C CNN
+F 2 "" H 5400 5000 50  0000 C CNN
+F 3 "" H 5400 5000 50  0000 C CNN
+	1    5400 5000
+	1    0    0    -1
+$EndComp
+Wire Wire Line
+	5400 4400 5400 5000
 $EndSCHEMATC
