File: hardware/desklight_panel.kicad_pcb (KiCad board)
At the start: 2 copper layers, 100 x 100 mm, 256 parts, among them IC1 ATTINY10-TS, P1 AVR_TPI, P2 Pwr5V1500mA, P3 WS2812_CON, SW1 Rotary_Encoder_Switch

Commit message: forward-port PCB to current kicad, include EC11 step model
Connections:
- net /~RESET renamed /~{RESET}
Other:
- net class Default removed
